Commit message: tricylinder
manifold mesh made with openscad. 2 models :(

File: models/tricylinder.urdf (robot description, URDF)
Before this commit: robot tricylinder, 1 links, 0 joints
Links:
- link tricylinderLink: geometry collision mesh filename=tricylinder_manifold.obj scale=1 1 1; visual mesh filename=tricylinder.obj scale=1 1 1
